File: pcb/seeeduino-xiao-breakout/seeeduino-xiao-breakout.kicad_sch (KiCad schematic)
At the start: 19 parts, among them J1 Conn_01x01_hole, J10 Conn_01x01_hole, J11 Conn_01x01_hole, J12 Conn_01x01_hole, J13 Conn_01x01_hole, J14 Conn_01x01_hole, J2 Conn_01x01_hole, J3 Conn_01x01_hole, J4 Conn_01x01_hole, J5 Conn_01x01_hole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

Commit message: increase power indicator resistor values
The previous resistors made the LEDs far brighter than they needed to be
Parts:
- R1: value 220 -> 470
- R2: value 100 -> 200

Commit message: create bom for pcb
Parts:
- D1, D2: Digikey Part # (none) -> 160-1169-1-ND; Part # (none) -> LTST-C150GKT
- J1, J10, J11, J12, J13, J14, J2, J3, J4, J5, J6, J7, J8, J9: Digikey Part # (none) -> N/A; Part # (none) -> N/A
- R1: value 470 -> 620; Digikey Part # (none) -> RMCF1206JT620RCT-ND; Part # (none) -> RMCF1206JT620R
- R2: value 200 -> 270; Digikey Part # (none) -> RMCF1206JT270RCT-ND; Part # (none) -> RMCF1206JT270R
- U1: Digikey Part # (none) -> 1597-102010328-ND; Part # (none) -> 102010328
